File: moon_knight_v2_left/moon_knight_v2_left.kicad_pcb (KiCad board)
At the start: 2 copper layers, 149.4 x 97.1 mm, 104 parts, among them U1 TRRS, U2 74HCT1G125GW

Commit message: Fixes
Parts:
- removed U1: TRRS, ScottoKeebs_Components:TRRS_PJ-320A
- removed U2: 74HCT1G125GW, Package_TO_SOT_SMD:SOT-23-5
- added J1: AudioJack4, PCM_marbastlib-xp-various:CON_MJ-4PP-9_Reversible, F.Cu at (166.9, 64.7)
- R1, R2: value 100R -> R
- moved R3 13.9 mm to (150.6, 34.2), turned to 180 degrees
- moved C23 2.81 mm to (163.8, 41.1)
- moved C24 2.81 mm to (163.8, 45.4)
- moved C25 2.81 mm to (163.7, 49.9)
- moved R1 2.58 mm to (155.4, 62.9), turned to 0 degrees
- moved R2 2.56 mm to (155.4, 66.2), turned to 0 degrees
- moved H7 2.00 mm to (158.0, 72.0)
Connections:
- MCU1 pad 4: GND -> 5V
- MCU1 pad 5: LED_IN_STEP -> LED_IN
Routing:
- net 5V: track 656.4 -> 678.8 mm, vias 40 -> 42
- net Net-(LED1-DIN): track 23.3 -> 4.43 mm, vias 2 -> 0
- net LED_IN: track 3.46 -> 15.4 mm
- net Col4: track 129.1 -> 138.5 mm
- net Col5: track 112.0 -> 121.0 mm
- net GND: track 9.89 -> 3.16 mm, vias 22 -> 23
- net LED_IN_STEP: track 6.03 -> 0.00 mm, vias 1 -> 0
- net TRRS_RX: track 27.1 -> 32.4 mm
- net TRRS_TX: track 27.0 -> 30.3 mm
- net Net-(J1-PadR1): track 11.5 -> 13.9 mm
- net Net-(D12-A): track 4.38 -> 6.43 mm
- net Col3: track 139.4 -> 141.3 mm
- net Net-(LED20-DOUT): track 24.1 -> 26.0 mm
- net Net-(LED21-DOUT): track 24.0 -> 22.1 mm, vias 0 -> 2
- net Net-(D8-A): track 3.84 -> 5.39 mm
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