File: moon_knight_v2_right/moon_knight_v2_right.kicad_pcb (KiCad board)
At the start: 2 copper layers, 149.4 x 97.1 mm, 104 parts, among them U1 TRRS, U2 74HCT1G125GW

Commit message: Fixes
Parts:
- removed U1: TRRS, PCM_marbastlib-xp-various:CON_MJ-4PP-9_Reversible
- removed U2: 74HCT1G125GW, Package_TO_SOT_SMD:SOT-23-5
- added J1: AudioJack4, PCM_marbastlib-xp-various:CON_MJ-4PP-9_Reversible, F.Cu at (66.5, 78.7)
- R3: value 47R -> 100R
- moved R3 8.90 mm to (82.7, 47.3), turned to 0 degrees
- moved R2 2.79 mm to (77.6, 77.1), turned to 0 degrees
- moved R1 2.57 mm to (77.6, 80.4), turned to 0 degrees
- moved H7 2.00 mm to (75.4, 85.8)
Connections:
- MCU1 pad 16: Col2 -> TRRS_TX
- MCU1 pad 17: Row1 -> TRRS_RX
- MCU1 pad 18: Col1 -> Col2
- MCU1 pad 19: TRRS_TX -> Row3
- MCU1 pad 20: TRRS_RX -> Row2
- MCU1 pad 21: Row3 -> Col0
- MCU1 pad 22: Row2 -> Col1
- MCU1 pad 23: Col0 -> Row1
- MCU1 pad 4: HANDEDNESS -> GND
- MCU1 pad 5: LED_IN_STEP -> LED_IN
- R1 pad 1: TRRS_TX -> Net-(J1-PadR2)
- R1 pad 2: Net-(U1-RING1) -> TRRS_RX
- R2 pad 1: TRRS_RX -> Net-(J1-PadR1)
- R2 pad 2: Net-(U1-RING2) -> TRRS_TX
Routing:
- net 5V: track 750.5 -> 709.3 mm, vias 38 -> 34
- net LED_IN: track 3.71 -> 23.8 mm, vias 0 -> 1
- net Net-(J1-PadR2): track 0.00 -> 16.8 mm
- net Net-(J1-PadR1): track 0.00 -> 12.4 mm
- net LED_IN_STEP: track 12.1 -> 0.00 mm, vias 1 -> 0
- net Row2: track 128.7 -> 140.4 mm, vias 0 -> 2
- net Net-(LED1-DIN): track 14.2 -> 3.67 mm
- net Col2: track 143.1 -> 152.5 mm
- net Net-(U1-RING2): track 9.22 -> 0.00 mm
- net Row3: track 124.1 -> 130.0 mm
- net Row1: track 117.6 -> 123.5 mm
- net TRRS_TX: track 13.7 -> 17.7 mm, vias 0 -> 1
- net Col1: track 126.3 -> 129.7 mm
- net GND: track 6.06 -> 9.16 mm, vias 15 -> 16
- net Col5: track 82.6 -> 80.4 mm
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