File: moon_knight_v2_right/moon_knight_v2_right.kicad_sch (KiCad schematic)
At the start: 104 parts, among them U1 TRRS, U2 74HCT1G125GW

Commit message: Fixes
Parts:
- removed R1, R2: 100R, Resistor_SMD:R_1206_3216Metric_Pad1.30x1.75mm_HandSolder, symbol ScottoKeebs:Placeholder_Resistor
- removed U1: TRRS, ScottoKeebs_Components:TRRS_PJ-320A, symbol ScottoKeebs:Placeholder_TRRS
- removed U2: 74HCT1G125GW, Package_TO_SOT_SMD:SOT-23-5, symbol 74xGxx:SN74LVC1G125DBV
- added J1: AudioJack4, PCM_marbastlib-xp-various:CON_MJ-4PP-9_Reversible, symbol Connector_Audio:AudioJack4
- added R1, R2: 100R, Resistor_SMD:R_1206_3216Metric_Pad1.30x1.75mm_HandSolder, symbol Device:R
- R3: value 47R -> 100R
Connections:
- net HANDEDNESS is gone; now on net GND: MCU1.4 (P29)
- net LED_IN_STEP is gone; now on net LED_IN: MCU1.5 (P28)
- net 5V: now also J1.T
- net Col0: now also MCU1.21 (P11); no longer MCU1.23 (P9)
- net Col1: now also MCU1.22 (P10); no longer MCU1.18 (P8)
- net Col2: now also MCU1.18 (P8); no longer MCU1.16 (P6)
- net GND: now also J1.S
- net Row1: now also MCU1.23 (P9); no longer MCU1.17 (P7)
- net Row2: now also MCU1.20 (P12); no longer MCU1.22 (P10)
- net Row3: now also MCU1.19 (P13); no longer MCU1.21 (P11)
- net TRRS_RX: now also MCU1.17 (P7), R1.2; no longer MCU1.20 (P12)
- net TRRS_TX: now also MCU1.16 (P6), R2.2; no longer MCU1.19 (P13)
- new net: J1.R1, R2.1
- new net: J1.R2, R1.1
