File: moon_knight_v3/moon_knight_v3.kicad_pcb (KiCad board)
At the start: 2 copper layers, 0 parts

Commit message: some commits
Parts:
- added C1: 0.1µF, Capacitor_SMD:C_1206_3216Metric, B.Cu at (132.0, 30.0)
- added C10: 0.1µF, Capacitor_SMD:C_1206_3216Metric, B.Cu at (115.5, 47.3)
- added C11: 0.1µF, Capacitor_SMD:C_1206_3216Metric, B.Cu at (133.5, 48.8)
- added C12: 0.1µF, Capacitor_SMD:C_1206_3216Metric, B.Cu at (150.6, 51.4)
- added C13: 0.1µF, Capacitor_SMD:C_1206_3216Metric, B.Cu at (133.7, 66.1)
- added C14: 0.1µF, Capacitor_SMD:C_1206_3216Metric, B.Cu at (115.7, 64.6)
- added C15: 0.1µF, Capacitor_SMD:C_1206_3216Metric, B.Cu at (97.7, 61.9)
- added C16: 0.1µF, Capacitor_SMD:C_1206_3216Metric, B.Cu at (79.6, 65.4)
- added C17: 0.1µF, Capacitor_SMD:C_1206_3216Metric, B.Cu at (62.0, 65.8)
- added C18: 0.1µF, Capacitor_SMD:C_1206_3216Metric, B.Cu at (46.2, 67.1)
- added C19: 0.1µF, Capacitor_SMD:C_1206_3216Metric, B.Cu at (125.0, 82.0)
- added C2: 0.1µF, Capacitor_SMD:C_1206_3216Metric, B.Cu at (115.7, 30.6)
- added C20: 0.1µF, Capacitor_SMD:C_1206_3216Metric, B.Cu at (145.6, 86.4)
- added C21: 0.1µF, Capacitor_SMD:C_1206_3216Metric, B.Cu at (155.7, 99.2)
- added C3: 0.1µF, Capacitor_SMD:C_1206_3216Metric, B.Cu at (97.6, 30.2)
- added C4: 0.1µF, Capacitor_SMD:C_1206_3216Metric, B.Cu at (79.7, 33.1)
- added C5: 0.1µF, Capacitor_SMD:C_1206_3216Metric, B.Cu at (61.6, 38.3)
- added C6: 0.1µF, Capacitor_SMD:C_1206_3216Metric, B.Cu at (46.2, 33.7)
- added C7: 0.1µF, Capacitor_SMD:C_1206_3216Metric, B.Cu at (60.8, 50.7)
- added C8: 0.1µF, Capacitor_SMD:C_1206_3216Metric, B.Cu at (78.8, 50.7)
- added C9: 0.1µF, Capacitor_SMD:C_1206_3216Metric, B.Cu at (95.4, 49.2)
- added CH1: choc_v1_SW_HS, PCM_marbastlib-choc:SW_choc_v1_HS_CPG135001S30_1u, B.Cu at (142.6, 36.8)
- added CH10: choc_v1_SW_HS, PCM_marbastlib-choc:SW_choc_v1_HS_CPG135001S30_1u, B.Cu at (106.6, 49.3)
- added CH11: choc_v1_SW_HS, PCM_marbastlib-choc:SW_choc_v1_HS_CPG135001S30_1u, B.Cu at (124.6, 52.3)
- added CH12: choc_v1_SW_HS, PCM_marbastlib-choc:SW_choc_v1_HS_CPG135001S30_1u, B.Cu at (142.6, 53.8)
- added CH13: choc_v1_SW_HS, PCM_marbastlib-choc:SW_choc_v1_HS_CPG135001S30_1u, B.Cu at (142.6, 70.8)
- added CH14: choc_v1_SW_HS, PCM_marbastlib-choc:SW_choc_v1_HS_CPG135001S30_1u, B.Cu at (124.6, 69.3)
- added CH15: choc_v1_SW_HS, PCM_marbastlib-choc:SW_choc_v1_HS_CPG135001S30_1u, B.Cu at (106.6, 66.3)
- added CH16: choc_v1_SW_HS, PCM_marbastlib-choc:SW_choc_v1_HS_CPG135001S30_1u, B.Cu at (88.6, 69.3)
- added CH17: choc_v1_SW_HS, PCM_marbastlib-choc:SW_choc_v1_HS_CPG135001S30_1u, B.Cu at (70.6, 72.3)
- added CH18: choc_v1_SW_HS, PCM_marbastlib-choc:SW_choc_v1_HS_CPG135001S30_1u, B.Cu at (52.6, 72.3)
- added CH19: choc_v1_SW_HS, PCM_marbastlib-choc:SW_choc_v1_HS_CPG135001S30_1u, B.Cu at (116.1, 87.0)
- added CH2: choc_v1_SW_HS, PCM_marbastlib-choc:SW_choc_v1_HS_CPG135001S30_1u, B.Cu at (124.6, 35.3)
- added CH20: choc_v1_SW_HS, PCM_marbastlib-choc:SW_choc_v1_HS_CPG135001S30_1u, B.Cu at (135.8, 89.1)
- added CH21: choc_v1_SW_HS, PCM_marbastlib-choc:SW_choc_v1_HS_CPG135001S30_1.5u, B.Cu at (156.2, 90.4)
- added CH3: choc_v1_SW_HS, PCM_marbastlib-choc:SW_choc_v1_HS_CPG135001S30_1u, B.Cu at (106.6, 32.3)
- added CH4: choc_v1_SW_HS, PCM_marbastlib-choc:SW_choc_v1_HS_CPG135001S30_1u, B.Cu at (88.6, 35.3)
- added CH5: choc_v1_SW_HS, PCM_marbastlib-choc:SW_choc_v1_HS_CPG135001S30_1u, B.Cu at (70.6, 38.3)
- added CH6: choc_v1_SW_HS, PCM_marbastlib-choc:SW_choc_v1_HS_CPG135001S30_1u, B.Cu at (52.6, 38.3)
- added CH7: choc_v1_SW_HS, PCM_marbastlib-choc:SW_choc_v1_HS_CPG135001S30_1u, B.Cu at (52.6, 55.3)
- added CH8: choc_v1_SW_HS, PCM_marbastlib-choc:SW_choc_v1_HS_CPG135001S30_1u, B.Cu at (70.6, 55.3)
- added CH9: choc_v1_SW_HS, PCM_marbastlib-choc:SW_choc_v1_HS_CPG135001S30_1u, B.Cu at (88.6, 52.3)
- added D1: 1N4148W, ScottoKeebs_Components:Diode_SOD-123, B.Cu at (145.7, 37.5)
- added D10: 1N4148W, ScottoKeebs_Components:Diode_SOD-123, B.Cu at (109.8, 50.3)
- added D11: 1N4148W, ScottoKeebs_Components:Diode_SOD-123, B.Cu at (127.8, 52.9)
- added D12: 1N4148W, ScottoKeebs_Components:Diode_SOD-123, B.Cu at (145.9, 54.4)
- added D13: 1N4148W, ScottoKeebs_Components:Diode_SOD-123, B.Cu at (145.7, 71.4)
- added D14: 1N4148W, ScottoKeebs_Components:Diode_SOD-123, B.Cu at (127.8, 70.0)
- added D15: 1N4148W, ScottoKeebs_Components:Diode_SOD-123, B.Cu at (109.8, 66.9)
- added D16: 1N4148W, ScottoKeebs_Components:Diode_SOD-123, B.Cu at (91.9, 69.8)
- added D17: 1N4148W, ScottoKeebs_Components:Diode_SOD-123, B.Cu at (73.8, 73.2)
- added D18: 1N4148W, ScottoKeebs_Components:Diode_SOD-123, B.Cu at (55.8, 73.1)
- added D19: 1N4148W, ScottoKeebs_Components:Diode_SOD-123, B.Cu at (119.3, 88.0)
- added D2: 1N4148W, ScottoKeebs_Components:Diode_SOD-123, B.Cu at (127.8, 36.6)
- added D20: 1N4148W, ScottoKeebs_Components:Diode_SOD-123, B.Cu at (138.8, 90.2)
- added D21: 1N4148W, ScottoKeebs_Components:Diode_SOD-123, B.Cu at (154.8, 93.3)
- added D3: 1N4148W, ScottoKeebs_Components:Diode_SOD-123, B.Cu at (109.8, 33.0)
- added D4: 1N4148W, ScottoKeebs_Components:Diode_SOD-123, B.Cu at (91.8, 35.8)
- added D5: 1N4148W, ScottoKeebs_Components:Diode_SOD-123, B.Cu at (73.8, 39.1)
- added D6: 1N4148W, ScottoKeebs_Components:Diode_SOD-123, B.Cu at (55.8, 39.2)
- added D7: 1N4148W, ScottoKeebs_Components:Diode_SOD-123, B.Cu at (55.8, 55.8)
- added D8: 1N4148W, ScottoKeebs_Components:Diode_SOD-123, B.Cu at (73.7, 56.4)
- added D9: 1N4148W, ScottoKeebs_Components:Diode_SOD-123, B.Cu at (91.9, 52.9)
- added H1: MountingHole, MountingHole:MountingHole_2.2mm_M2, F.Cu at (61.6, 33.3)
- added H2: MountingHole, MountingHole:MountingHole_2.2mm_M2, F.Cu at (133.6, 33.3)
- added H3: MountingHole, MountingHole:MountingHole_2.2mm_M2, F.Cu at (97.6, 46.0)
- added H4: MountingHole, MountingHole:MountingHole_2.2mm_M2, F.Cu at (61.6, 70.3)
- added H5: MountingHole, MountingHole:MountingHole_2.2mm_M2, F.Cu at (148.4, 81.4)
- added H6: MountingHole, MountingHole:MountingHole_2.2mm_M2, F.Cu at (167.7, 71.2)
- added H7: MountingHole, MountingHole:MountingHole_2.2mm_M2, F.Cu at (157.7, 71.2)
- added J1: AudioJack4, PCM_marbastlib-xp-various:CON_MJ-4PP-9_Reversible, F.Cu at (164.6, 63.7)
- added LED1: SK6812MINI-E, PCM_marbastlib-various:LED_6028R, B.Cu at (142.6, 31.8)
- added LED10: SK6812MINI-E, PCM_marbastlib-various:LED_6028R, B.Cu at (106.6, 44.3)
- added LED11: SK6812MINI-E, PCM_marbastlib-various:LED_6028R, B.Cu at (124.6, 47.3)
- added LED12: SK6812MINI-E, PCM_marbastlib-various:LED_6028R, B.Cu at (142.6, 48.8)
- added LED13: SK6812MINI-E, PCM_marbastlib-various:LED_6028R, B.Cu at (142.6, 65.8)
- added LED14: SK6812MINI-E, PCM_marbastlib-various:LED_6028R, B.Cu at (124.6, 64.3)
- added LED15: SK6812MINI-E, PCM_marbastlib-various:LED_6028R, B.Cu at (106.6, 61.3)
- added LED16: SK6812MINI-E, PCM_marbastlib-various:LED_6028R, B.Cu at (88.6, 64.3)
- added LED17: SK6812MINI-E, PCM_marbastlib-various:LED_6028R, B.Cu at (70.6, 67.3)
- added LED18: SK6812MINI-E, PCM_marbastlib-various:LED_6028R, B.Cu at (52.6, 67.3)
- added LED19: SK6812MINI-E, PCM_marbastlib-various:LED_6028R, B.Cu at (116.1, 82.0)
- added LED2: SK6812MINI-E, PCM_marbastlib-various:LED_6028R, B.Cu at (124.6, 30.3)
- added LED20: SK6812MINI-E, PCM_marbastlib-various:LED_6028R, B.Cu at (136.8, 84.2)
- added LED21: SK6812MINI-E, PCM_marbastlib-various:LED_6028R, B.Cu at (160.7, 92.5)
- added LED3: SK6812MINI-E, PCM_marbastlib-various:LED_6028R, B.Cu at (106.6, 27.3)
- added LED4: SK6812MINI-E, PCM_marbastlib-various:LED_6028R, B.Cu at (88.6, 30.3)
- added LED5: SK6812MINI-E, PCM_marbastlib-various:LED_6028R, B.Cu at (70.6, 33.3)
- added LED6: SK6812MINI-E, PCM_marbastlib-various:LED_6028R, B.Cu at (52.6, 33.3)
- added LED7: SK6812MINI-E, PCM_marbastlib-various:LED_6028R, B.Cu at (52.6, 50.3)
- added LED8: SK6812MINI-E, PCM_marbastlib-various:LED_6028R, B.Cu at (70.6, 50.3)
- added LED9: SK6812MINI-E, PCM_marbastlib-various:LED_6028R, B.Cu at (88.6, 47.3)
- added MCU1: RP2040-Matrix, PCM_marbastlib-xp-promicroish:RP2040-Matrix_AH, F.Cu at (161.0, 45.4)
- added R1: R, Resistor_SMD:R_1206_3216Metric_Pad1.30x1.75mm_HandSolder, B.Cu at (153.1, 66.6)
- added R2: R, Resistor_SMD:R_1206_3216Metric_Pad1.30x1.75mm_HandSolder, B.Cu at (150.3, 66.6)
- added R3: 47R, Resistor_SMD:R_1206_3216Metric_Pad1.30x1.75mm_HandSolder, B.Cu at (158.7, 41.1)
Routing:
- net 5V: track 0.00 -> 576.9 mm, vias 0 -> 35
- net Col0: track 0.00 -> 162.0 mm
- net Col1: track 0.00 -> 142.5 mm
- net Row2: track 0.00 -> 129.6 mm
- net Col3: track 0.00 -> 124.7 mm
- net Col2: track 0.00 -> 120.7 mm
- net Row0: track 0.00 -> 118.5 mm
- net Row1: track 0.00 -> 115.6 mm
- net Row3: track 0.00 -> 100.6 mm
- net Col4: track 0.00 -> 99.9 mm, vias 0 -> 2
- net Col5: track 0.00 -> 78.3 mm
- net Net-(LED18-DOUT): track 0.00 -> 78.2 mm, vias 0 -> 2
- net Net-(LED20-DOUT): track 0.00 -> 29.5 mm, vias 0 -> 2
- net TRRS_TX: track 0.00 -> 29.3 mm, vias 0 -> 1
- net TRRS_RX: track 0.00 -> 27.9 mm, vias 0 -> 1
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- added copper zone on B.Cu, net GND
- added copper zone on F.Cu, net GND
Other:
- board outline added: 126.7 x 82.4 mm
- board text added: "Designed By Deepanshu Jain"
