File: moon_knight_v4/moon_knight_v4.kicad_pcb (KiCad board)
At the start: 2 copper layers, 128.8 x 82.2 mm, 98 parts, among them J1 AudioJack4, J2 OLED_128x32, SW1 SW_PUSH, U1 Sea-Picro

Commit message: v4 keeb
Parts:
- added H8: MountingHole, MountingHole:MountingHole_2.2mm_M2, F.Cu at (134.1, 71.8)
- added H9: MountingHole, MountingHole:MountingHole_2.2mm_M2, F.Cu at (98.2, 80.5)
- moved H3 26.2 mm to (98.1, 34.7)
- moved C13 1.65 mm to (134.1, 67.4)
- moved H7 0.61 mm to (155.6, 73.3)
Routing:
- net SCL: track 33.6 -> 23.7 mm
- net SDA: track 38.9 -> 31.2 mm, vias 1 -> 4
- net 5V: track 560.9 -> 568.1 mm
- net Row3: track 112.6 -> 108.9 mm
- net Col0: track 172.6 -> 170.9 mm
- net Net-(J1-PadR2): track 28.1 -> 29.6 mm
- net Row1: track 134.9 -> 133.6 mm, vias 1 -> 3
- net Net-(LED15-DOUT): track 13.2 -> 14.4 mm, vias 0 -> 4
- net TRRS_RX: track 17.7 -> 18.4 mm
- net Net-(LED3-DOUT): track 13.6 -> 14.2 mm, vias 0 -> 2
- net Net-(J1-PadR1): track 29.0 -> 29.6 mm
- net Net-(LED14-DOUT): track 14.4 -> 14.9 mm, vias 0 -> 4
- net Net-(LED16-DOUT): track 12.9 -> 13.1 mm, vias 0 -> 2
- net Row2: vias 1 -> 5
- net GND: vias 26 -> 17

Commit message: v4
Parts:
- removed J2: OLED_128x32, kleeb_display:OLED-128x32
- removed SW1: SW_PUSH, Button_Switch_SMD:SW_SPST_TS-1088-xR020
- R1, R2: moved to F.Cu
- U1: value Sea-Picro -> RP2040-Matrix; footprint josh-module:Sea-Picro_EXT_Module_Flipped -> PCM_marbastlib-xp-promicroish:RP2040-Matrix_AH
- moved R2 19.6 mm to (155.8, 69.5), turned to 180 degrees
- moved H9 16.5 mm to (98.0, 64.0)
- moved R1 14.3 mm to (155.8, 66.5), turned to 180 degrees
- moved H2 12.0 mm to (134.1, 48.4)
- moved H1 11.2 mm to (62.1, 49.9)
- moved H3 10.3 mm to (98.1, 45.0)
- moved J1 7.62 mm to (166.2, 65.4)
- moved H4 6.50 mm to (62.1, 66.8)
- moved H8 6.44 mm to (134.1, 65.3)
- moved H6 5.88 mm to (168.0, 73.5)
- moved R3 5.16 mm to (162.9, 45.5), turned to 180 degrees
- moved C1 4.60 mm to (135.3, 35.2), turned to -90 degrees
- moved C17 3.04 mm to (63.1, 71.8), turned to -90 degrees
- moved C13 3.01 mm to (135.3, 70.2)
- moved C10 2.86 mm to (114.8, 47.7), turned to -90 degrees
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Connections:
- U1 pad 1: unconnected-(U1-USB+-Pad1) -> 5V
- U1 pad 10: Row3 -> unconnected-(U1-P0-Pad10)
- U1 pad 11: Row2 -> Col5
- U1 pad 12: Col0 -> Col4
- U1 pad 13: Col1 -> Col3
- U1 pad 14: unconnected-(U1-IO12-Pad14) -> Col2
- U1 pad 15: unconnected-(U1-IO13-Pad15) -> Col1
- U1 pad 16: unconnected-(U1-IO14-Pad16) -> TRRS_TX
- U1 pad 17: unconnected-(U1-IO15-Pad17) -> TRRS_RX
- U1 pad 18: unconnected-(U1-IO16-Pad18) -> Col0
- U1 pad 19: Col2 -> unconnected-(U1-P13-Pad19)
- U1 pad 2: TRRS_TX -> GND
- U1 pad 20: Col3 -> unconnected-(U1-P12-Pad20)
- U1 pad 21: Col4 -> unconnected-(U1-P11-Pad21)
- U1 pad 22: Col5 -> unconnected-(U1-P10-Pad22)
- U1 pad 3: TRRS_RX -> unconnected-(U1-3V3-Pad3)
- U1 pad 4: GND -> unconnected-(U1-P29-Pad4)
- U1 pad 5: GND -> LED_IN
- U1 pad 6: SDA -> Row0
- U1 pad 7: SCL -> Row1
- U1 pad 8: Row0 -> Row3
- U1 pad 9: Row1 -> Row2
Routing:
- net Col3: track 122.8 -> 161.2 mm, vias 1 -> 2
- net Col5: track 78.4 -> 116.1 mm, vias 3 -> 0
- net Col2: track 114.0 -> 146.7 mm, vias 1 -> 2
- net SDA: track 31.2 -> 0.00 mm, vias 4 -> 0
- net Col4: track 108.8 -> 138.2 mm, vias 1 -> 2
- net Row1: track 133.6 -> 109.5 mm, vias 3 -> 0
- net Row3: track 108.9 -> 85.0 mm, vias 3 -> 2
- net SCL: track 23.7 -> 0.00 mm, vias 1 -> 0
- net Net-(J1-PadR1): track 29.6 -> 8.13 mm
- net Row2: track 137.6 -> 117.7 mm, vias 5 -> 0
- net 5V: track 568.1 -> 585.9 mm, vias 29 -> 22
- net Net-(J1-PadR2): track 29.6 -> 13.2 mm
- net RST: track 12.5 -> 0.00 mm
- net Col1: track 155.3 -> 166.8 mm
- net Row0: track 132.3 -> 123.4 mm, vias 1 -> 0
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Other:
- board size 128.8 x 82.2 mm -> 129.3 x 82.2 mm
- board text added: "Deepanshu Jain"
