File: moon_knight_v4_right/moon_knight_v4_right.kicad_pcb (KiCad board)
At the start: 2 copper layers, 128.8 x 82.2 mm, 98 parts, among them J1 AudioJack4, J2 OLED_128x32, SW1 SW_PUSH, U1 Sea-Picro

Commit message: v4
Parts:
- removed J2: OLED_128x32, kleeb_display:OLED-128x32
- removed SW1: SW_PUSH, Button_Switch_SMD:SW_SPST_TS-1088-xR020
- added H8: MountingHole, MountingHole:MountingHole_2.2mm_M2, B.Cu at (114.3, 103.2)
- added H9: MountingHole, MountingHole:MountingHole_2.2mm_M2, B.Cu at (150.4, 101.8)
- R1, R2: moved to F.Cu
- U1: value Sea-Picro -> RP2040-Matrix; footprint josh-module:Sea-Picro_EXT_Module_Flipped -> PCM_marbastlib-xp-promicroish:RP2040-Matrix_AH
- moved R1 67.6 mm to (91.5, 102.7)
- moved C21 64.1 mm to (88.6, 139.3), turned to 180 degrees
- moved R2 63.6 mm to (91.5, 100.2)
- moved C1 62.6 mm to (113.4, 73.1), turned to 90 degrees
- moved H2 60.8 mm to (114.3, 86.2)
- moved H1 60.1 mm to (186.3, 87.7)
- moved H3 59.4 mm to (150.3, 82.8)
- moved C17 55.1 mm to (186.5, 109.7)
- moved C15 54.4 mm to (150.5, 107.8)
- moved C7 53.9 mm to (189.1, 92.5)
- moved C5 53.7 mm to (185.1, 74.5)
- moved C2 53.2 mm to (131.2, 71.5), turned to -90 degrees
- moved C13 53.1 mm to (113.3, 107.9), turned to 90 degrees
- moved C12 52.9 mm to (99.1, 90.0)
- moved C4 52.9 mm to (167.1, 71.5), turned to 90 degrees
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Connections:
- U1 pad 1: unconnected-(U1-USB+-Pad1) -> 5V
- U1 pad 10: Row3 -> unconnected-(U1-P0-Pad10)
- U1 pad 11: Row2 -> Col5
- U1 pad 12: Col1 -> Col4
- U1 pad 13: Col0 -> Col3
- U1 pad 14: unconnected-(U1-IO12-Pad14) -> Col2
- U1 pad 15: unconnected-(U1-IO13-Pad15) -> Col1
- U1 pad 16: unconnected-(U1-IO14-Pad16) -> TRRS_TX
- U1 pad 17: unconnected-(U1-IO15-Pad17) -> TRRS_RX
- U1 pad 18: unconnected-(U1-IO16-Pad18) -> Col0
- U1 pad 19: Col2 -> unconnected-(U1-P13-Pad19)
- U1 pad 2: TRRS_TX -> GND
- U1 pad 20: Col3 -> unconnected-(U1-P12-Pad20)
- U1 pad 21: Col4 -> unconnected-(U1-P11-Pad21)
- U1 pad 22: Col5 -> unconnected-(U1-P10-Pad22)
- U1 pad 3: TRRS_RX -> unconnected-(U1-3V3-Pad3)
- U1 pad 4: GND -> unconnected-(U1-P29-Pad4)
- U1 pad 5: GND -> LED_IN
- U1 pad 6: SDA -> Row0
- U1 pad 7: SCL -> Row1
- U1 pad 8: Row0 -> Row3
- U1 pad 9: Row1 -> Row2
Routing:
- net Row3: track 88.2 -> 30.6 mm, vias 7 -> 0
- net Net-(D19-A): track 4.30 -> 54.8 mm
- net Col3: track 158.0 -> 110.9 mm, vias 2 -> 0
- net Net-(D20-A): track 4.35 -> 39.2 mm
- net SDA: track 32.1 -> 0.00 mm, vias 1 -> 0
- net Col2: track 131.4 -> 99.5 mm, vias 2 -> 0
- net SCL: track 30.1 -> 0.00 mm, vias 1 -> 0
- net Row0: track 116.4 -> 142.1 mm
- net Net-(J1-PadR1): track 28.0 -> 4.18 mm, vias 2 -> 0
- net Col5: track 82.7 -> 59.7 mm, vias 1 -> 0
- net Col1: track 143.8 -> 121.3 mm, vias 2 -> 0
- net Col4: track 111.2 -> 92.7 mm, vias 1 -> 0
- net Col0: track 158.3 -> 141.4 mm, vias 2 -> 0
- net Net-(J1-PadR2): track 25.0 -> 8.47 mm, vias 1 -> 0
- net Row1: track 113.6 -> 130.1 mm, vias 11 -> 0
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Other:
- board size 128.8 x 82.2 mm -> 129.3 x 82.2 mm
